File: Triac Switch/TriacSwitch.brd (EAGLE design)
At the start: 63.2 x 63.5 mm, 14 parts, among them T2 BT136

Commit message: Added Pinout to UD001 (Vishay) after successful test
Parts:
- added R6: 270R / 560R, resistor:0207/10
- added S1: SWITCH-MOMENTARY-2PTH, SparkFun-Electromechanical:TACTILE-PTH
- moved F1 33.0 mm to (41.9, 12.7), turned to 180 degrees
Connections:
- removed net N$10: OK1.2, R1.2
- new net N$5: R6.1, S1.3
- new net N$8: OK1.1, R1.2, R6.2
- net GND: now also OK1.2
- net VCC: now also S1.1; no longer OK1.1
Routing:
- net 220V_LIVE: track 57.6 -> 0.00 mm
- net N$1: track 161.5 -> 178.5 mm
- net N$10: track 13.0 -> 0.00 mm
- net N$2: track 10.5 -> 0.00 mm
- net GND: track 11.2 -> 20.6 mm
- net VCC: track 37.9 -> 36.6 mm
